File: canhat.kicad_pcb (KiCad board)
At the start: 2 copper layers, 65 x 30 mm, 42 parts, among them J1 Raspberry_Pi_2_3, J2 CAN In/Out/GND, J3 GPIO, J5 12V, U1 MCP2515-xSO, U2 SN65HVDA541, U3 AT24C32-SSHM, U4 AP63205, Y1 16MHz

Commit message: initial commit
Other:
- board text added: "CAN HAT V8 for Raspberry Pi © 2023 onitake"
- board text removed: "CAN HAT V8 for Raspberry Pi © 2020 onitake"
